File: cad_files/mm8d.sch (KiCad schematic (older format))
At the start: 51 parts

Commit message: 210109
Parts:
- removed D? (x6): D, symbol D
- removed JP?: Jumper_NO_Small, symbol Jumper_NO_Small
- removed Q? (x4): Q_NPN_CBE, symbol Q_NPN_CBE
- removed R? (x10): R, symbol R
- added C1, C2: 100n, Capacitors_THT:C_Rect_L7_W2.5_P5, symbol C
- added C3: 470u, Capacitors_THT:C_Radial_D8_L11.5_P3.5, symbol CP
- added C4: 47u, Capacitors_THT:C_Radial_D8_L11.5_P3.5, symbol CP
- added D10, D11, D12, D13, D14, D15, D16, D17, D18, D5, D6, D7, D8: LED, LEDs:LED-3MM, symbol LED
- added D2, D20, D21, D22, D3, D4, D9: 1N4001, Diodes_THT:Diode_DO-41_SOD81_Horizontal_RM10, symbol D
- added JP1: Jumper_NC_Small, Socket_Strips:Socket_Strip_Straight_1x02, symbol Jumper_NC_Small
- added JP2: Jumper_NO_Small, Socket_Strips:Socket_Strip_Straight_1x02, symbol Jumper_NO_Small
- added Q5, Q6, Q7, Q8: BC548C, TO_SOT_Packages_THT:TO-92_Rugged, symbol Q_NPN_CBE
- added R10, R11, R12, R9: 4.7k, Discret:R4, symbol R
- added R14, R15, R17, R18, R19, R20, R21: 1.5k, Discret:R4, symbol R
- added R16: 3,6k, Discret:R4, symbol R
- added R2, R3, R4: 9.1k, Discret:R4, symbol R
- added U5: 74LS14, Housings_DIP:DIP-14_W7.62mm_LongPads, symbol 74LS14
- added U6: 74LS05, Housings_DIP:DIP-14_W7.62mm_LongPads, symbol 74LS05
- D1, D19: renamed from D?; value D -> 1N4001; footprint (none) -> Diodes_THT:Diode_DO-41_SOD81_Horizontal_RM10
- J1, J10: renamed from J?; footprint (none) -> Connectors:bornier5
- J2, J3, J4, J5: renamed from J?; footprint (none) -> Connectors:bornier4
- J6, J7, J8, J9: renamed from J?; footprint (none) -> Connectors:bornier3
- K1, K2, K3, K4: renamed from K?; value Relay_LEG-5 -> LEG-5
- Q1, Q2, Q3, Q4: renamed from Q?; value Q_NPN_CBE -> BC548C; footprint (none) -> TO_SOT_Packages_THT:TO-92_Rugged
- R1: renamed from R?; value R -> 9.1k; footprint (none) -> Discret:R4
- R13: renamed from R?; value R -> 1.5k; footprint (none) -> Discret:R4
- R5, R6, R7, R8: renamed from R?; value R -> 4.7k; footprint (none) -> Discret:R4
- U1, U2, U3, U4: renamed from U?; footprint DIP-6 -> Housings_DIP:DIP-6_W7.62mm_LongPads
Connections:
- net at J1.2: now also R2.2
- net at J1.3: now also R3.2
- net at J1.4: now also R4.2
- net at D1.2 (A), J1.5, U1.2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: now also D2.2 (A), D3.2 (A), D4.2 (A)
- net at D1.1 (K), R1.1: now also D5.2 (A); no longer U1.1
- net GNDD: now reaches U1.4, U2.4, U3.4, U4.4
- net GNDD: now also J10.5, J3.2, J3.3, Q1.3 (E), Q2.3 (E), Q3.3 (E), Q4.3 (E), C1.2, C2.2, C3.2, C4.2, D9.2 (A), Q5.3 (E), Q6.3 (E), Q7.3 (E), Q8.3 (E), R16.2, U5.11, U5.13, U6.11, U6.13
- net at R5.2, U1.5: now also U5.1; no longer J2.1
- net at U2.1: now also D6.1 (K)
- net at R6.2, U2.5: now also U5.3; no longer J2.2
- net at U3.1: now also D7.1 (K)
- net at R7.2, U3.5: now also U5.5; no longer J2.3
- net at U4.1: now also D8.1 (K)
- net at R8.2, U4.5: now also U5.9; no longer J2.4
- net at J3.1, R5.1, R6.1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: now also D19.1 (K), K1.1 (Coil), K2.1 (Coil), K3.1 (Coil), K4.1 (Coil), C1.1, C2.1, C3.1, D10.2 (A), D20.1 (K), D21.1 (K), D22.1 (K), D9.1 (K), JP1.2
- net at J10.1: now also Q5.1 (C)
- net at J10.2: now also Q6.1 (C)
- net at J10.3: now also Q7.1 (C)
- net at J10.4: now also Q8.1 (C)
- net at J4.1: now also R13.1; no longer R13.2
- net at J4.2: now also R14.1
- net at J4.3: now also R15.1
- net at J4.4: now also R17.1
- net at J5.1: now also R18.1
- net at J5.2: now also R19.1
- net at J5.3: now also R20.1
- net at J5.4: now also R21.1
- net at Q1.2 (B): now also D11.1 (K); no longer R13.1
- net at Q2.2 (B): now also D12.1 (K)
- net at Q3.2 (B): now also D13.1 (K)
- net at Q4.2 (B): now also D14.1 (K)
- net at K4.2 (Coil), Q4.1 (C): now also D22.2 (A)
- net at K3.2 (Coil), Q3.1 (C): now also D21.2 (A)
- net at K2.2 (Coil), Q2.1 (C): now also D20.2 (A)
- new net: D5.1 (K), U1.1
- new net: C4.1, J3.4, JP2.2
- new net: J2.1, R9.2, U6.2
- new net: J2.2, R10.2, U6.4
- new net: J2.3, R11.2, U6.6
- new net: J2.4, R12.2, U6.8
- new net: D11.2 (A), R13.2
- new net: D2.1 (K), D6.2 (A), R2.1
- new net: D3.1 (K), D7.2 (A), R3.1
- new net: D4.1 (K), D8.2 (A), R4.1
- new net: U5.2, U6.1
- new net: U5.4, U6.3
- new net: U5.6, U6.5
- new net: U5.8, U6.9
- new net: D12.2 (A), R14.2
- new net: D13.2 (A), R15.2
- new net: D14.2 (A), R17.2
- new net: D15.2 (A), R18.2
- new net: D16.2 (A), R19.2
- new net: D17.2 (A), R20.2
- new net: D18.2 (A), R21.2
- new net: JP1.1, JP2.1, R10.1, R11.1, R12.1, R9.1
- new net: D10.1 (K), R16.1
- new net: D15.1 (K), Q5.2 (B)
- new net: D16.1 (K), Q6.2 (B)
- new net: D17.1 (K), Q7.2 (B)
- new net: D18.1 (K), Q8.2 (B)
- new net GND: U5.7 (GND), U5.7 (GND), U5.7 (GND), U5.7 (GND), U5.7 (GND), U5.7 (GND), U6.7 (GND), U6.7 (GND), U6.7 (GND), U6.7 (GND), U6.7 (GND), U6.7 (GND)
- new net VCC: U5.14 (VCC), U5.14 (VCC), U5.14 (VCC), U5.14 (VCC), U5.14 (VCC), U5.14 (VCC), U6.14 (VCC), U6.14 (VCC), U6.14 (VCC), U6.14 (VCC), U6.14 (VCC), U6.14 (VCC)
- no-connect marks 4 -> 8
Other:
- moved on the sheet: D1, D19, J1, J10, J2, J3, J4, J5, J6, J7, J8, J9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

Commit message: 210325
Parts:
- added R10, R12, R14, R16: 1k, Discret:R5, symbol R
- C4: value 47u -> 4.7u; footprint Capacitors_THT:C_Radial_D8_L11.5_P3.5 -> Capacitors_THT:C_Radial_D5_L11_P2.5
- K1, K2, K3, K4: footprint (none) -> Discret:relay_leg
- R1, R2, R3, R4, R5, R6, R7, R8, R9: footprint Discret:R4 -> Discret:R5
- R11: renamed from R10; footprint Discret:R4 -> Discret:R5
- R13: renamed from R11; footprint Discret:R4 -> Discret:R5
- R15: renamed from R12; footprint Discret:R4 -> Discret:R5
- R17: renamed from R13; footprint Discret:R4 -> Discret:R5
- R18: renamed from R14; footprint Discret:R4 -> Discret:R5
- R19: renamed from R15; footprint Discret:R4 -> Discret:R5
- R20: renamed from R17; footprint Discret:R4 -> Discret:R5
- R21: renamed from R16; footprint Discret:R4 -> Discret:R5
- R22: renamed from R18; footprint Discret:R4 -> Discret:R5
- R23: renamed from R19; footprint Discret:R4 -> Discret:R5
- R24: renamed from R20; footprint Discret:R4 -> Discret:R5
- R25: renamed from R21; footprint Discret:R4 -> Discret:R5
- renumbered C2 to C1, C1 to C2, Q5 to Q2, Q2 to Q3, Q6 to Q4, Q3 to Q5, Q7 to Q6, Q4 to Q7
Connections:
- net GNDD is gone; now on net GND: C1.2, C2.2, C3.2, C4.2, D9.2 (A), J10.5, J3.2, J3.3, Q1.3 (E), Q2.3 (E), Q3.3 (E), Q4.3 (E), Q5.3 (E), Q6.3 (E), Q7.3 (E), Q8.3 (E), R21.2, U1.4, U2.4, U3.4, U4.4, U5.11, U5.13, U6.11, U6.13
- net VCC: now also C1.1, C2.1, C3.1, D10.2 (A), D19.1 (K), D20.1 (K), D21.1 (K), D22.1 (K), D9.1 (K), J3.1, JP1.2, K1.1 (Coil), K2.1 (Coil), K3.1 (Coil), K4.1 (Coil), R5.1, R6.1, R7.1, R8.1
- net at R9.2, U6.2: now also R10.2; no longer J2.1
- net at R11.2, U6.4: now also R12.2; no longer J2.2
- net at R13.2, U6.6: now also R14.2; no longer J2.3
- net at R15.2, U6.8: now also R16.2; no longer J2.4
- new net: J2.1, R10.1
- new net: J2.2, R12.1
- new net: J2.3, R14.1
- new net: J2.4, R16.1
Other:
- moved on the sheet: C1, C2, C3, C4, D1, D10, D11, D12, D13, D14, D15, D16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

Commit message: 210325
Parts:
- C1, C2: footprint Capacitors_THT:C_Rect_L7_W2.5_P5 -> Capacitors_THT:C_Rect_L7.0mm_W2.5mm_P5.00mm
- C3: footprint Capacitors_THT:C_Radial_D8_L11.5_P3.5 -> Capacitors_THT:CP_Radial_D8.0mm_P3.50mm
- C4: footprint Capacitors_THT:C_Radial_D5_L11_P2.5 -> Capacitors_THT:CP_Radial_D5.0mm_P2.50mm
- D1, D19, D2, D20, D21, D22, D3, D4, D9: footprint Diodes_THT:Diode_DO-41_SOD81_Horizontal_RM10 -> Diodes_THT:D_DO-41_SOD81_P10.16mm_Horizontal
- D10, D11, D12, D13, D14, D15, D16, D17, D18, D5, D6, D7, D8: footprint LEDs:LED-3MM -> LEDs:LED_D3.0mm
- JP1, JP2: footprint Socket_Strips:Socket_Strip_Straight_1x02 -> Socket_Strips:Socket_Strip_Straight_1x02_Pitch2.54mm
- K1, K2, K3, K4: footprint Discret:relay_leg -> relay_lg:relay_leg
- R1, R10, R11, R12, R13, R14, R15, R16, R17, R18, R19, R2, R20, R21, R22, R23, R24, R25, R3, R4, R5, R6, R7, R8, R9: footprint Discret:R5 -> Resistors_THT:R_Axial_DIN0411_L9.9mm_D3.6mm_P12.70mm_Horizontal

Commit message: 210326
Connections:
- net at J7.2: now also K2.3 (Common); no longer K2.4 (NC)
- net at J7.3: now also K2.4 (NC); no longer K2.3 (Common)
- net at J9.2: now also K4.3 (Common); no longer K4.4 (NC)
- net at J9.3: now also K4.4 (NC); no longer K4.3 (Common)
- net at J8.2: now also K3.3 (Common); no longer K3.4 (NC)
- net at J8.3: now also K3.4 (NC); no longer K3.3 (Common)
- net at J6.2: now also K1.3 (Common); no longer K1.4 (NC)
- net at J6.3: now also K1.4 (NC); no longer K1.3 (Common)
Changed lines of the file:
@@
 	13850 4225 13850 4325
 Wire Wire Line
-	13850 4325 14450 4325
-Wire Wire Line
 	13900 3925 13900 3875
 Wire Wire Line
 	13900 3875 14100 3875
 Wire Wire Line
-	14100 3875 14100 4125
-Wire Wire Line
-	14100 4125 14450 4125
+	14100 3875 14100 4325
 Wire Wire Line
 	14450 3925 14200 3925
@@
 	13850 4875 13850 4975
 Wire Wire Line
-	13850 4975 14450 4975
-Wire Wire Line
 	13900 4575 13900 4525
 Wire Wire Line
 	13900 4525 14100 4525
 Wire Wire Line
-	14100 4525 14100 4775
-Wire Wire Line
-	14100 4775 14450 4775
+	14100 4525 14100 4975
 Wire Wire Line
 	14450 4575 14200 4575
@@
 	13850 5525 13850 5625
 Wire Wire Line
-	13850 5625 14450 5625
-Wire Wire Line
 	13900 5225 13900 5175
 Wire Wire Line
 	13900 5175 14100 5175
 Wire Wire Line
-	14100 5175 14100 5425
-Wire Wire Line
-	14100 5425 14450 5425
+	14100 5175 14100 5625
 Wire Wire Line
 	14450 5225 14200 5225
@@
 	13850 6175 13850 6275
 Wire Wire Line
-	13850 6275 14450 6275
-Wire Wire Line
 	13900 5875 13900 5825
 Wire Wire Line
 	13900 5825 14100 5825
 Wire Wire Line
-	14100 5825 14100 6075
-Wire Wire Line
-	14100 6075 14450 6075
+	14100 5825 14100 6275
 Wire Wire Line
 	14450 5875 14200 5875
@@
 	5575 4900 5475 4900
 Connection ~ 5475 4900
+Wire Wire Line
+	14100 4325 14450 4325
+Wire Wire Line
+	14100 4975 14450 4975
+Wire Wire Line
+	14100 5625 14450 5625
+Wire Wire Line
+	14100 6275 14450 6275
+Wire Wire Line
+	14450 6075 14000 6075
+Wire Wire Line
+	14000 6075 14000 6275
+Wire Wire Line
+	14000 6275 13850 6275
+Wire Wire Line
+	13850 5625 14000 5625
+Wire Wire Line
+	14000 5625 14000 5425
+Wire Wire Line
+	14000 5425 14450 5425
+Wire Wire Line
+	13850 4975 14000 4975
+Wire Wire Line
+	14000 4975 14000 4775
+Wire Wire Line
+	14000 4775 14450 4775
+Wire Wire Line
+	13850 4325 14000 4325
+Wire Wire Line
+	14000 4325 14000 4125
+Wire Wire Line
+	14000 4125 14450 4125
 $EndSCHEMATC
