File: cad_files/mm8d.sch (KiCad schematic (older format))
At the start: 81 parts, among them J1 Screw_Terminal_1x05, J10 Screw_Terminal_1x05, J2 Screw_Terminal_1x04, J3 Screw_Terminal_1x04, J4 Screw_Terminal_1x04, J5 Screw_Terminal_1x04, J6 Screw_Terminal_1x03, J7 Screw_Terminal_1x03, J8 Screw_Terminal_1x03, J9 Screw_Terminal_1x03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

Commit message: 210327
Parts:
- added D23: LED, LEDs:LED_D3.0mm, symbol LED
- added R26: 620, Resistors_THT:R_Axial_DIN0411_L9.9mm_D3.6mm_P12.70mm_Horizontal, symbol R
- R10, R12, R14, R16: value 1k -> 750
- R17, R18, R19, R20, R22, R23, R24, R25: value 1.5k -> 620
- R21: value 3,6k -> 1k
Connections:
- net GND: now also R26.2
- net at C4.1, J3.4, JP2.2: now also D23.2 (A)
- new net: D23.1 (K), R26.1
Other:
- note added: "+3.3V"
- note added: "+5V"
