File: cad_files/mm8d.sch (KiCad schematic (older format))
At the start: 83 parts, among them J1 Screw_Terminal_1x05, J10 Screw_Terminal_1x05, J2 Screw_Terminal_1x04, J3 Screw_Terminal_1x04, J4 Screw_Terminal_1x04, J5 Screw_Terminal_1x04, J6 Screw_Terminal_1x03, J7 Screw_Terminal_1x03, J8 Screw_Terminal_1x03, J9 Screw_Terminal_1x03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

Commit message: 220330
Parts:
- R1, R2, R3, R4: value 9.1k -> 3.9k
Changed lines of the file:
@@
 P 2425 5175
 F 0 "R1" V 2525 5175 50  0000 C CNN
-F 1 "9.1k" V 2325 5175 50  0000 C CNN
+F 1 "3.9k" V 2325 5175 50  0000 C CNN
 F 2 "Resistors_THT:R_Axial_DIN0411_L9.9mm_D3.6mm_P12.70mm_Horizontal" V 2355 5175 50  0001 C CNN
 F 3 "" H 2425 5175 50  0000 C CNN
@@
 P 2425 5650
 F 0 "R2" V 2525 5650 50  0000 C CNN
-F 1 "9.1k" V 2325 5650 50  0000 C CNN
+F 1 "3.9k" V 2325 5650 50  0000 C CNN
 F 2 "Resistors_THT:R_Axial_DIN0411_L9.9mm_D3.6mm_P12.70mm_Horizontal" V 2355 5650 50  0001 C CNN
 F 3 "" H 2425 5650 50  0000 C CNN
@@
 P 2425 6125
 F 0 "R3" V 2525 6125 50  0000 C CNN
-F 1 "9.1k" V 2325 6125 50  0000 C CNN
+F 1 "3.9k" V 2325 6125 50  0000 C CNN
 F 2 "Resistors_THT:R_Axial_DIN0411_L9.9mm_D3.6mm_P12.70mm_Horizontal" V 2355 6125 50  0001 C CNN
 F 3 "" H 2425 6125 50  0000 C CNN
@@
 P 2425 6600
 F 0 "R4" V 2525 6600 50  0000 C CNN
-F 1 "9.1k" V 2325 6600 50  0000 C CNN
+F 1 "3.9k" V 2325 6600 50  0000 C CNN
 F 2 "Resistors_THT:R_Axial_DIN0411_L9.9mm_D3.6mm_P12.70mm_Horizontal" V 2355 6600 50  0001 C CNN
 F 3 "" H 2425 6600 50  0000 C CNN
