File: cad_files/mm8d.kicad_pcb (KiCad board)
At the start: 2 copper layers, 81 parts, among them J1 Screw_Terminal_1x05, J10 Screw_Terminal_1x05, J2 Screw_Terminal_1x04, J3 Screw_Terminal_1x04, J4 Screw_Terminal_1x04, J5 Screw_Terminal_1x04, J6 Screw_Terminal_1x03, J7 Screw_Terminal_1x03, J8 Screw_Terminal_1x03, J9 Screw_Terminal_1x03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

Commit message: 210326
Parts:
- moved D22 153.6 mm to (260.4, 92.5), turned to 180 degrees
- moved D21 136.7 mm to (242.8, 92.5), turned to 180 degrees
- moved D20 119.9 mm to (225.3, 92.5), turned to 180 degrees
- moved R20 118.7 mm to (250.2, 81.0)
- moved D14 115.0 mm to (262.4, 88.9), turned to 90 degrees
- moved K4 108.0 mm to (256.5, 105.9), turned to 270 degrees
- moved J9 104.4 mm to (251.5, 122.4)
- moved Q7 103.1 mm to (250.2, 88.1)
- moved R19 102.8 mm to (232.7, 81.0)
- moved J3 102.4 mm to (51.3, 72.9)
- moved D13 97.9 mm to (245.1, 88.9), turned to 90 degrees
- moved C3 93.1 mm to (55.6, 98.6)
- moved K3 90.5 mm to (239.0, 105.9), turned to 270 degrees
- moved R8 89.6 mm to (59.2, 111.5), turned to 270 degrees
- moved R25 88.8 mm to (189.7, 80.8), turned to 270 degrees
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Connections:
- K1 pad 3: Net-(J6-Pad3) -> Net-(J6-Pad2)
- K1 pad 4: Net-(J6-Pad2) -> Net-(J6-Pad3)
- K2 pad 3: Net-(J7-Pad3) -> Net-(J7-Pad2)
- K2 pad 4: Net-(J7-Pad2) -> Net-(J7-Pad3)
- K3 pad 3: Net-(J8-Pad3) -> Net-(J8-Pad2)
- K3 pad 4: Net-(J8-Pad2) -> Net-(J8-Pad3)
- K4 pad 3: Net-(J9-Pad3) -> Net-(J9-Pad2)
- K4 pad 4: Net-(J9-Pad2) -> Net-(J9-Pad3)
Routing:
- net Net-(D1-Pad2): track 0.00 -> 46.6 mm
- net Net-(J4-Pad1): track 0.00 -> 32.1 mm
- net Net-(D2-Pad1): track 0.00 -> 26.1 mm
- net Net-(D3-Pad1): track 0.00 -> 25.9 mm
- net VCC: track 0.00 -> 24.8 mm
- net Net-(J7-Pad2): track 0.00 -> 24.7 mm
- net Net-(J6-Pad2): track 0.00 -> 24.7 mm
- net Net-(J8-Pad2): track 0.00 -> 24.7 mm
- net Net-(J9-Pad2): track 0.00 -> 24.7 mm
- net Net-(R11-Pad2): track 0.00 -> 20.6 mm
- net Net-(R13-Pad2): track 0.00 -> 20.3 mm
- net Net-(J4-Pad4): track 0.00 -> 19.1 mm
- net Net-(J4-Pad2): track 0.00 -> 17.7 mm
- net Net-(J10-Pad4): track 0.00 -> 15.9 mm
- net Net-(D8-Pad1): track 0.00 -> 15.8 mm
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
Commit message: 210305
Parts:
- moved C1 26.8 mm to (127.8, 98.6)
- moved C2 26.8 mm to (144.3, 98.6)
- moved D10 24.9 mm to (46.2, 87.1), turned to 180 degrees
- moved R5 23.9 mm to (66.0, 101.9), turned to 270 degrees
- moved R6 23.9 mm to (61.0, 101.9), turned to 270 degrees
- moved R7 23.9 mm to (55.9, 101.9), turned to 270 degrees
- moved C4 17.1 mm to (65.8, 81.8), turned to 180 degrees
- moved C3 13.0 mm to (66.3, 91.2), turned to 180 degrees
- moved R8 12.6 mm to (51.1, 101.9)
- moved JP2 10.5 mm to (69.1, 74.7), turned to 180 degrees
- moved R21 9.45 mm to (43.7, 93.5)
- moved D22 7.64 mm to (252.7, 93.0)
- moved K4 7.64 mm to (248.9, 106.4)
- moved D1 7.64 mm to (79.5, 94.0)
- moved D11 7.64 mm to (202.1, 89.3)
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Routing:
- net GND: track 0.00 -> 496.1 mm
- net VCC: track 24.8 -> 444.5 mm
- net Net-(R8-Pad2): track 0.00 -> 88.0 mm
- net Net-(JP1-Pad1): track 10.2 -> 94.6 mm
- net Net-(R7-Pad2): track 0.00 -> 75.5 mm
- net Net-(D1-Pad2): track 46.6 -> 117.6 mm
- net Net-(R6-Pad2): track 0.00 -> 68.9 mm
- net Net-(R5-Pad2): track 0.00 -> 66.4 mm
- net Net-(R13-Pad2): track 20.3 -> 62.1 mm
- net Net-(R10-Pad2): track 5.08 -> 43.0 mm
- net Net-(R15-Pad2): track 5.08 -> 36.3 mm
- net Net-(R11-Pad2): track 20.6 -> 50.8 mm
- net Net-(C4-Pad1): track 0.00 -> 20.6 mm
- net Net-(U5-Pad8): track 0.00 -> 17.7 mm
- net Net-(U5-Pad4): track 0.00 -> 17.7 mm
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Other:
- board outline added: 218.2 x 59.7 mm
