File: cad_files/mm8d.kicad_pcb (KiCad board)
At the start: 2 copper layers, 238.5 x 59.7 mm, 92 parts, among them J1 Screw_Terminal_1x05, J10 Screw_Terminal_1x05, J2 Screw_Terminal_1x04, J3 Screw_Terminal_1x04, J4 Screw_Terminal_1x04, J5 Screw_Terminal_1x04, J6 Screw_Terminal_1x03, J7 Screw_Terminal_1x03, J8 Screw_Terminal_1x03, J9 Screw_Terminal_1x03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

Commit message: 210327
Parts:
- added D23: LED, LEDs:LED_D3.0mm, F.Cu at (51.1, 86.6)
- added R26: 620, Resistors_THT:R_Axial_DIN0411_L9.9mm_D3.6mm_P12.70mm_Horizontal, F.Cu at (42.9, 101.3)
- R10, R12, R14, R16: value 1k -> 750
- R17, R18, R19, R20, R22, R23, R24, R25: value 1.5k -> 620
- R21: value 3,6k -> 1k
- moved R8 0.13 mm to (47.9, 101.3)
Routing:
- net Net-(D23-Pad1): track 0.00 -> 19.3 mm
- net Net-(C4-Pad1): track 20.6 -> 34.0 mm
- net GND: track 489.3 -> 487.1 mm
- net VCC: track 444.5 -> 443.2 mm
