File: cad_files/mm8d.kicad_pcb (KiCad board)
At the start: 2 copper layers, 238.5 x 59.7 mm, 94 parts, among them J1 Screw_Terminal_1x05, J10 Screw_Terminal_1x05, J2 Screw_Terminal_1x04, J3 Screw_Terminal_1x04, J4 Screw_Terminal_1x04, J5 Screw_Terminal_1x04, J6 Screw_Terminal_1x03, J7 Screw_Terminal_1x03, J8 Screw_Terminal_1x03, J9 Screw_Terminal_1x03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

Commit message: 220330
Parts:
- R1, R2, R3, R4: value 9.1k -> 3.9k
Changed lines of the file:
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@@
       (effects (font (size 1 1) (thickness 0.15)))
     )
-    (fp_text value 9.1k (at 6.35 2.86 90) (layer F.Fab)
+    (fp_text value 3.9k (at 6.35 2.86 90) (layer F.Fab)
       (effects (font (size 1 1) (thickness 0.15)))
     )
@@
       (effects (font (size 1 1) (thickness 0.15)))
     )
-    (fp_text value 9.1k (at 6.35 2.86 90) (layer F.Fab)
+    (fp_text value 3.9k (at 6.35 2.86 90) (layer F.Fab)
       (effects (font (size 1 1) (thickness 0.15)))
     )
@@
       (effects (font (size 1 1) (thickness 0.15)))
     )
-    (fp_text value 9.1k (at 6.35 2.86 90) (layer F.Fab)
+    (fp_text value 3.9k (at 6.35 2.86 90) (layer F.Fab)
       (effects (font (size 1 1) (thickness 0.15)))
     )
@@
       (effects (font (size 1 1) (thickness 0.15)))
     )
-    (fp_text value 9.1k (at 6.35 2.86 90) (layer F.Fab)
-      (effects (font (size 1 1) (thickness 0.15)))
-    )
+    (fp_text value 3.9k (at 6.35 2.86 90) (layer F.Fab)
+      (effects (font (size 1 1) (thickness 0.15)))
+    )
